Commit message: Fix parameter names and update inertial macros in inertial_macros.xacro and robot_core.xacro

File: description/inertial_macros.xacro (robot description, xacro)
@@ -1,18 +1,18 @@
 <?xml version="1.0"?>
 <robot xmlns:xacro="http://www.ros.org/wiki/xacro">
-    <xacro:macro name="inertial_sphere" params="mass raduis *origin">
+    <xacro:macro name="inertial_sphere" params="mass radius *origin">
         <inertial>
             <mass value="${mass}"/>
-            <inertia ixx = "${(2/5)*mass*(raduis*radius)}" ixy ="0.0" ixz = "0.0"
-                iyy = "${(2/5)*mass*(raduis*radius)}" iyz = "0.0"
-                izz = "${(2/5)*mass*(raduis*radius)}"/>
+            <inertia ixx = "${(2/5)*mass*(radius*radius)}" ixy ="0.0" ixz = "0.0"
+                iyy = "${(2/5)*mass*(radius*radius)}" iyz = "0.0"
+                izz = "${(2/5)*mass*(radius*radius)}"/>
         </inertial>
     </xacro:macro>
-    <xacro:macro name = "inertial_box" params = "mass size *origin">
+    <xacro:macro name = "inertial_box" params = "mass x y z *origin">
     <inertial>
         <mass value = "${mass}"/>
-        <inertia ixx ="${(1/12)*mass * radius (y*y + z*z)}" ixy ="0.0" ixz = "0.0"
-                iyy = "${(1/12)*mass * radius (x*x + z*z)}" iyz = "0.0"
-                izz = "${(1/12)*mass * radius (x*x + y*y)}"/>
+        <inertia ixx ="${(1/12)*mass * (y*y + z*z)}" ixy ="0.0" ixz = "0.0"
+                iyy = "${(1/12)*mass * (x*x + z*z)}" iyz = "0.0"
+                izz = "${(1/12)*mass * (x*x + y*y)}"/>
     </inertial>
     </xacro:macro>

File: description/robot_core.xacro (robot description, xacro)
@@ -1,4 +1,5 @@
 <?xml version="1.0"?>
 <robot xmlns:xacro="http://www.ros.org/wiki/xacro">
+    <xacro:include filename="inertial_macros.xacro"/>
     <material name = "white">
         <color rgba="1 1 1 1"/>
@@ -64,5 +65,5 @@
             </geometry>
         </collision>
-        <xacro:inertial_cylinder mass = "0.1" length="0.04" radius= " 0.05">
+        <xacro:inertial_cylinder mass = "0.1" height="0.04" radius= " 0.05">
             <origin xyz = "0 0 0" rpy = "0 0 0"/>
         </xacro:inertial_cylinder>
@@ -87,5 +88,5 @@
             </geometry>
         </collision>
-        <xacro:inertial_cylinder mass = "0.1" length="0.04" radius= " 0.05">
+        <xacro:inertial_cylinder mass = "0.1" height="0.04" radius= " 0.05">
             <origin xyz = "0 0 0" rpy = "0 0 0"/>
         </xacro:inertial_cylinder>
