Commit message: Fix typos in robot_control.xarco, enhance material definitions in robot_core.xacro, and update launch_sim.launch.py for improved simulation parameters

File: description/robot_core.xacro (robot description, xacro)
@@ -2,67 +2,74 @@
 <robot xmlns:xacro="http://www.ros.org/wiki/xacro">
     <xacro:include filename="inertial_macros.xacro"/>
-    <material name = "white">
-        <color rgba="1 1 1 1"/>
+    <!-- Define PBR Materials -->
+    <material name="blue">
+        <color rgba="0.2 0.2 1 1"/>
+        <pbr>
+            <albedo>0.2 0.2 1 1</albedo>
+            <roughness>0.5</roughness>
+            <metalness>0.1</metalness>
+        </pbr>
     </material>
-    <material name = "ishaan">
-        <color rgba="0 0 0 1"/>
+    <material name="orange">
+        <color rgba="1 0.3 0.2 1"/>
+        <pbr>
+            <albedo>1 0.3 0.2 1</albedo>
+            <roughness>0.5</roughness>
+            <metalness>0.2</metalness>
+        </pbr>
     </material>
-    <material name = "blue">
-        <color rgba="0.2 0.2 1 1"/>
-    </material>
-    <material name = "orange">
-        <color rgba="1 0.3 0.2 1"/>
-    </material>
-    <!--BASE LINK-->
-    <link name = "base_link">
-           <inertial>
-            <origin xyz = "0 0 0" rpy = "0 0 0"/>
-            <mass value = "1"/>
-            <inertia ixx = "0.1" ixy = "0" ixz = "0" iyy = "0.1" iyz = "0" izz = "0.1"/>
-           </inertial>
-    </link>
-    <gazebo reference="base_link">
-        <material>Gazebo/White</material>
-    </gazebo>
-    <!--CHASSIS-->
-    <joint name="chassis_joint" type="fixed">
-        <parent link = "base_link"/>
-        <child link = "chassis"/>
-        <origin xyz = "-0.1 0 0"/>
-    </joint>
-    <link name = "chassis">
+    <!-- BASE LINK -->
+    <link name="base_link">
+        <inertial>
+            <origin xyz="0 0 3" rpy="0 0 0"/>
+            <mass value="1"/>
+            <inertia ixx="0.1" ixy="0" ixz="0" iyy="0.1" iyz="0" izz="0.1"/>
+        </inertial>
         <visual>
-           <geometry>
-               <box size = "0.3 0.3 0.15"/>
+            <geometry>
+                <box size="0.1 0.1 0.1"/>
             </geometry>
-            <material name = "blue"/>
-             <origin xyz = "0.15 0 0.075"/>
         </visual>
         <collision>
-           <geometry>
-               <box size = "0.3 0.3 0.15"/>
+            <geometry>
+                <box size="0.1 0.1 0.1"/>
             </geometry>
-             <origin xyz = "0.15 0 0.075"/>
         </collision>
-        <xacro:inertial_box mass = "0.5" x="0.3" y= " 0.3" z = "0.15">
-            <origin xyz = "0.15 0 0.075" rpy = "0 0 0"/>
+    </link>
+    <!-- CHASSIS -->
+    <joint name="chassis_joint" type="fixed">
+        <parent link="base_link"/>
+        <child link="chassis"/>
+        <origin xyz="-0.1 0 0"/>
+    </joint>
+    <link name="chassis">
+        <visual>
+            <geometry>
+                <box size="0.3 0.3 0.15"/>
+            </geometry>
+            <material name="blue"/>
+        </visual>
+        <collision>
+            <geometry>
+                <box size="0.3 0.3 0.15"/>
+            </geometry>
+        </collision>
+        <xacro:inertial_box mass = "0.5" x="0.3" y = "0.3" z = "0.15">
+            <origin xyz="0.15 0 0.075" rpy="0 0 0"/>
         </xacro:inertial_box>
     </link>
-    <gazebo reference="chassis">
-        <material>Gazebo/Blue</material>
-    </gazebo>
-    <!--LEFT WHEEL LINK-->
+    <!-- LEFT WHEEL -->
     <joint name="left_wheel_joint" type="continuous">
-        <parent link = "base_link"/>
-        <child link = "left_wheel"/>
-        <origin xyz = "0 0.175 0" rpy = "-${pi/2} 0 0"/>
-        <axis xyz = "0 0 1"/>
+        <parent link="base_link"/>
+        <child link="left_wheel"/>
+        <origin xyz="0 0.175 -0.05" rpy="-${pi/2} 0 0"/>
+        <axis xyz="0 0 1"/>
     </joint>
-    <link name = "left_wheel">
+    <link name="left_wheel">
         <visual>
             <geometry>
                 <cylinder radius="0.05" length="0.04"/>
             </geometry>
-            <material name = "orange"/>
+            <material name="orange"/>
         </visual>
         <collision>
@@ -71,24 +78,21 @@
             </geometry>
         </collision>
-        <xacro:inertial_cylinder mass = "0.1" height="0.04" radius= " 0.05">
-            <origin xyz = "0 0 0" rpy = "0 0 0"/>
+        <xacro:inertial_cylinder mass="0.1" radius="0.05" height="0.04">
+            <origin xyz="0 0 0" rpy="0 0 0"/>
         </xacro:inertial_cylinder>
     </link>
-    <gazebo reference="left_wheel">
-        <material>Gazebo/Orange</material>
-    </gazebo>
-    <!--RIGHT WHEEL LINK-->
+    <!-- RIGHT WHEEL -->
     <joint name="right_wheel_joint" type="continuous">
-        <parent link = "base_link"/>
-        <child link = "right_wheel"/>
-        <origin xyz = "0 -0.175 0" rpy = "${pi/2} 0 0"/>
-        <axis xyz = "0 0 -1"/>
+        <parent link="base_link"/>
+        <child link="right_wheel"/>
+        <origin xyz="0 -0.175 -0.05" rpy="${pi/2} 0 0"/>
+        <axis xyz="0 0 -1"/>
     </joint>
-    <link name = "right_wheel">
+    <link name="right_wheel">
         <visual>
             <geometry>
                 <cylinder radius="0.05" length="0.04"/>
             </geometry>
-            <material name = "orange"/>
+            <material name="orange"/>
         </visual>
         <collision>
@@ -97,30 +101,29 @@
             </geometry>
         </collision>
-        <xacro:inertial_cylinder mass = "0.1" height="0.04" radius= " 0.05">
-            <origin xyz = "0 0 0" rpy = "0 0 0"/>
+        <xacro:inertial_cylinder mass="0.1" radius="0.05" height="0.04">
+            <origin xyz="0 0 0" rpy="0 0 0"/>
         </xacro:inertial_cylinder>
     </link>
-    <gazebo reference="right_wheel">
-        <material>Gazebo/Orange</material>
-    </gazebo>
-    <!--CASTER WHEEL LINK-->
-    <joint name = "caster_wheel_wheel" type = "fixed">
-        <parent link = "base_link"/>
-        <child link = "caster_wheel"/>
-        <origin xyz = "0.24 0 0" rpy = "0 0 0"/>
+    <!-- CASTER WHEEL -->
+    <joint name="caster_wheel_joint" type="fixed">
+        <parent link="chassis"/>
+        <child link="caster_wheel"/>
+        <origin xyz="-0.14 0 -0.05"/>
     </joint>
-    <link name = "caster_wheel">
+    <link name="caster_wheel">
         <visual>
             <geometry>
-                <sphere radius = "0.05"/>
+                <sphere radius="0.05"/>
             </geometry>
-            <material name = "ishaan"/>
+            <material name="orange"/>
         </visual>
-        <xacro:inertial_sphere mass = "0.1" radius= " 0.05">
-            <origin xyz = "0 0 0" rpy = "0 0 0"/>
+        <collision>
+            <geometry>
+                <sphere radius="0.05"/>
+            </geometry>
+        </collision>
+        <xacro:inertial_sphere mass="0.1" radius="0.05">
+            <origin xyz="0 0 0" rpy="0 0 0"/>
         </xacro:inertial_sphere>
     </link>
-    <gazebo reference="caster_wheel">
-        <material>Gazebo/Ishaan</material>
-    </gazebo>
 </robot>

Commit message: Fix base link origin in robot_core.xacro to correct simulation positioning

File: description/robot_core.xacro (robot description, xacro)
@@ -22,5 +22,5 @@
     <link name="base_link">
         <inertial>
-            <origin xyz="0 0 3" rpy="0 0 0"/>
+            <origin xyz="0 0 0" rpy="0 0 0"/>
             <mass value="1"/>
             <inertia ixx="0.1" ixy="0" ixz="0" iyy="0.1" iyz="0" izz="0.1"/>
