Commit message: Remove inertial_macros.xarco file

File: description/robot.urdf.xacro (robot description, xacro)
@@ -2,4 +2,4 @@
 <robot xmlns:xacro="http://www.ros.org/wiki/xacro"  name="robot">
     <!-- Example link -->
-    <xacro:include filename = "robot_core.xarco"/>
+    <xacro:include filename = "robot_core.xacro"/>
 </robot>

File: description/robot_core.xacro (robot description, xacro)
@@ -1,4 +1,4 @@
 <?xml version="1.0"?>
-<robot xmlns:xacro="http://www.ros.org/wiki/xacro" xmlns:xarco="http://www.ros.org/wiki/xacro">
+<robot xmlns:xacro="http://www.ros.org/wiki/xacro">
     <material name = "white">
         <color rgba="1 1 1 1"/>
@@ -15,4 +15,9 @@
     <!--BASE LINK-->
     <link name = "base_link">
+           <inertial>
+            <origin xyz = "0 0 0" rpy = "0 0 0"/>
+            <mass value = "1"/>
+            <inertia ixx = "0.1" ixy = "0" ixz = "0" iyy = "0.1" iyz = "0" izz = "0.1"/>
+           </inertial>
     </link>
     <!--CHASSIS-->
@@ -36,7 +41,7 @@
              <origin xyz = "0.15 0 0.075"/>
         </collision>
-        <xarco:inertial_box mass = "0.5" x="0.3" y= " 0.3" z = "0.15">
+        <xacro:inertial_box mass = "0.5" x="0.3" y= " 0.3" z = "0.15">
             <origin xyz = "0.15 0 0.075" rpy = "0 0 0"/>
-        </xarco:inertial_box>
+        </xacro:inertial_box>
     </link>
     <!--LEFT WHEEL LINK-->
@@ -59,7 +64,7 @@
             </geometry>
         </collision>
-        <xarco:inertial_cylinder mass = "0.1" length="0.04" radius= " 0.05">
+        <xacro:inertial_cylinder mass = "0.1" length="0.04" radius= " 0.05">
             <origin xyz = "0 0 0" rpy = "0 0 0"/>
-        </xarco:inertial_cylinder>
+        </xacro:inertial_cylinder>
     </link>
     <!--RIGHT WHEEL LINK-->
@@ -82,7 +87,7 @@
             </geometry>
         </collision>
-        <xarco:inertial_cylinder mass = "0.1" length="0.04" radius= " 0.05">
+        <xacro:inertial_cylinder mass = "0.1" length="0.04" radius= " 0.05">
             <origin xyz = "0 0 0" rpy = "0 0 0"/>
-        </xarco:inertial_cylinder>
+        </xacro:inertial_cylinder>
     </link>
     <!--CASTER WHEEL LINK-->
@@ -99,7 +104,7 @@
             <material name = "ishaan"/>
         </visual>
-        <xarco:inertial_sphere mass = "0.1" radius= " 0.05">
+        <xacro:inertial_sphere mass = "0.1" radius= " 0.05">
             <origin xyz = "0 0 0" rpy = "0 0 0"/>
-        </xarco:inertial_sphere>
+        </xacro:inertial_sphere>
     </link>
 </robot>

Commit message: Add robot_control.xarco and update robot_core.xacro with gazebo materials

File: description/robot.urdf.xacro (robot description, xacro)
@@ -3,3 +3,4 @@
     <!-- Example link -->
     <xacro:include filename = "robot_core.xacro"/>
+    <xacro:include filename = "robot_control.xarco"/>
 </robot>

File: description/robot_core.xacro (robot description, xacro)
@@ -22,4 +22,7 @@
            </inertial>
     </link>
+    <gazebo reference="base_link">
+        <material>Gazebo/White</material>
+    </gazebo>
     <!--CHASSIS-->
     <joint name="chassis_joint" type="fixed">
@@ -46,4 +49,7 @@
         </xacro:inertial_box>
     </link>
+    <gazebo reference="chassis">
+        <material>Gazebo/Blue</material>
+    </gazebo>
     <!--LEFT WHEEL LINK-->
     <joint name="left_wheel_joint" type="continuous">
@@ -69,4 +75,7 @@
         </xacro:inertial_cylinder>
     </link>
+    <gazebo reference="left_wheel">
+        <material>Gazebo/Orange</material>
+    </gazebo>
     <!--RIGHT WHEEL LINK-->
     <joint name="right_wheel_joint" type="continuous">
@@ -92,4 +101,7 @@
         </xacro:inertial_cylinder>
     </link>
+    <gazebo reference="right_wheel">
+        <material>Gazebo/Orange</material>
+    </gazebo>
     <!--CASTER WHEEL LINK-->
     <joint name = "caster_wheel_wheel" type = "fixed">
@@ -109,3 +121,6 @@
         </xacro:inertial_sphere>
     </link>
+    <gazebo reference="caster_wheel">
+        <material>Gazebo/Ishaan</material>
+    </gazebo>
 </robot>

Commit message: Update robot configuration: change SLAM mode to mapping, remove my_controllers.yaml, add robot_controllers.yaml, and enhance launch file for controller management

File: description/robot.urdf.xacro (robot description, xacro)
@@ -5,3 +5,4 @@
     <xacro:include filename = "gazebo_control.xacro"/>
     <xacro:include filename = "lidar.xacro"/>
+    <xacro:include filename = "ros2_control.xacro"/>
 </robot>

File: description/robot_core.xacro (robot description, xacro)
@@ -36,4 +36,11 @@
             </geometry>
         </collision>
+    </link>
+    <joint name="base_footprint_joint" type="fixed">
+        <parent link="base_link"/>
+        <child link="base_footprint"/>
+        <origin xyz="0 0 0"/>
+    </joint>
+    <link name = "base_footprint">
     </link>
     <!-- CHASSIS -->

File: description/ros2_control.xacro (robot description, xacro)
@@ -1,13 +1,12 @@
 <?xml version="1.0"?>
 <robot xmlns:xacro="http://www.ros.org/wiki/xacro">
-    <xacro:unless value="$(arg sim_mode)">
-        <ros2_control name="RealRobot" type="system">
+  <ros2_control name="RealRobot" type="system">
             <hardware>
-                <plugin>diffdrive_arduino/DiffDriveArduinoHardware</plugin>
+                <plugin>ros2_control_demo_example_2/DiffBotSystemHardware</plugin>
                 <param name="left_wheel_name">left_wheel_joint</param>
                 <param name="right_wheel_name">right_wheel_joint</param>
                 <param name="loop_rate">30</param>
-                <param name="device">/dev/ttyUSB0</param>
-                <param name="baud_rate">115200</param>
+                <param name="device">/dev/ttyACM0</param>
+                <param name="baud_rate">9600</param>
                 <param name="timeout_ms">1000</param>
                 <param name="enc_counts_per_rev">3436</param>
@@ -30,33 +29,3 @@
             </joint>
         </ros2_control>
-    </xacro:unless>
-    <!-- <xacro:if value="$(arg sim_mode)">
-        <ros2_control name="GazeboSystem" type="system">
-            <hardware>
-                <plugin>gz_ros2_control/GazeboSimSystem</plugin>
-            </hardware>
-            <joint name="left_wheel_joint">
-                <command_interface name="velocity">
-                    <param name="min">-10</param>
-                    <param name="max">10</param>
-                </command_interface>
-                <state_interface name="velocity"/>
-                <state_interface name="position"/>
-            </joint>
-            <joint name="right_wheel_joint">
-                <command_interface name="velocity">
-                    <param name="min">-10</param>
-                    <param name="max">10</param>
-                </command_interface>
-                <state_interface name="velocity"/>
-                <state_interface name="position"/>
-            </joint>
-        </ros2_control>
-    </xacro:if> -->
-    <gazebo>
-        <plugin name="gz_ros2_control::GazeboSimROS2ControlPlugin" filename="libgz_ros2_control-system.so">
-            <parameters>$(find my_bot)/config/my_controllers.yaml</parameters>
-            <!-- <parameters>$(find my_bot)/config/gaz_ros2_ctl_use_sim.yaml</parameters> -->
-        </plugin>
-    </gazebo>
 </robot>
